File: grad-cap-pcb/adder.kicad_sch (KiCad schematic)
At the start: 0 parts

Commit message: added many things
added: mux
counter
signal gen - still needs r1 and r2 values
power management
kicad symbol library - footprints not assigned
Parts:
- added R6, R7, R8, R9: 10K, symbol Device:R_Small_US
- added U4, U5: MC74HC73ADR2G, SOIC-14_NB_ONS, symbol MC74HC73ADR2G_JK-FLIPFLOP:MC74HC73ADR2G
Connections:
- new net: R6.2, U5.2 (RESET1), U5.3 (K1)
- new net: R8.2, U4.10 (K2), U4.14 (J1)
- new net: R7.2, U4.2 (RESET1), U4.3 (K1), U4.6 (RESET2), U4.7 (J2)
- new net: R9.2, U5.14 (J1)
- new net +3.3V: R6.1, R7.1, R8.1, R9.1, U4.4 (VCC), U5.4 (VCC)
- new net CLOCK1: U4.1 (CLOCK1)
- new net CLOCK2: U4.12 (Q1), U4.5 (CLOCK2)
- new net CLOCK3: U4.9 (Q2), U5.1 (CLOCK1)
- new net CLOCK4: U5.12 (Q1)
- new net GND: U4.11 (GND), U5.11 (GND), U5.6 (RESET2)
- no-connect marks 0 -> 8
Other:
- note added: "INPUT FROM 555"
