File: grad-cap-pcb/pulse_gen.kicad_sch (KiCad schematic)
At the start: 0 parts

Commit message: added many things
added: mux
counter
signal gen - still needs r1 and r2 values
power management
kicad symbol library - footprints not assigned
Parts:
- added C1: C_Small_US, symbol Device:C_Small_US
- added C2: C_Small, symbol Device:C_Small
- added R4, R5: R_Small_US, symbol Device:R_Small_US
- added U7: ICM7555xB, Package_SO:SOIC-8_3.9x4.9mm_P1.27mm, symbol Timer:ICM7555xB
Connections:
- new net: C2.1, U7.5 (CV)
- new net: R4.1, R5.2, U7.7 (DIS)
- new net: C1.1, R4.2, U7.2 (TR), U7.6 (THR)
- new net +3.3V: R5.1, U7.4 (R), U7.8 (VCC)
- new net CLOCK1: U7.3 (Q)
- new net GND: C1.2, C2.2, U7.1 (GND)
Other:
- note added: "CLOCK OUTPUT"
- note added: "R1"
- note added: "R2"
