File: grad-cap-pcb/grad-cap-pcb.kicad_pcb (KiCad board)
At the start: 4 copper layers, 339.4 x 339.4 mm, 205 parts, among them J1 B02B-XASK-1LFSN, T1 PHPT610035PKX, T2 PHPT610035PKX, T3 PHPT610035PKX, T4 PHPT610035PKX, T5 PHPT610035PKX, T6 PHPT610035PKX, T7 PHPT610035PKX, T8 PHPT610035PKX, U1 CD4072BM96, U10 CD74HC154M96, U2 CD4075BM96, U3 SN74AHCT32DBR, U4 MC74HC73ADR2G, U5 MC74HC73ADR2G, U6 SN74AHCT32DBR, U7 ICM7555xB, U8 SN74AHCT32DBR, U9 XC6220B211MR-G

Commit message: screw it were making it 8 frames, 16 is too mcuh
Parts:
- removed D103: LED, LED_SMD:LED_0603_1608Metric
- moved D107 1.87 mm to (287.0, 278.0)
- moved R13 0.71 mm to (259.5, 283.5)
- turned D12 to -90 degrees
- turned D141 to 90 degrees
- turned D9 to 67.5 degrees
Connections:
- D90 pad 2: /leds+mosfets/14or15 -> /leds+mosfets/frame14
- T1 pad 1: +2V2 -> +3.3V
- T1 pad 3: +2V2 -> +3.3V
- T2 pad 1: +2V2 -> +3.3V
- T2 pad 3: +2V2 -> +3.3V
- T3 pad 1: +2V2 -> +3.3V
- T3 pad 3: +2V2 -> +3.3V
- T4 pad 1: +2V2 -> +3.3V
- T4 pad 3: +2V2 -> +3.3V
- T5 pad 1: +2V2 -> +3.3V
- T5 pad 3: +2V2 -> +3.3V
- T6 pad 1: +2V2 -> +3.3V
- T6 pad 3: +2V2 -> +3.3V
- T7 pad 1: +2V2 -> +3.3V
- T7 pad 3: +2V2 -> +3.3V
- T8 pad 1: +2V2 -> +3.3V
- T8 pad 3: +2V2 -> +3.3V
- U9 pad 5: +2V2 -> +3.3V
Routing:
- net /leds+mosfets/frame4: track 0.00 -> 356.2 mm, vias 0 -> 7
- net /leds+mosfets/6or7: track 61.0 -> 413.0 mm, vias 0 -> 2
- net /leds+mosfets/frame15: track 0.00 -> 335.0 mm, vias 0 -> 4
- net /leds+mosfets/frame7: track 150.0 -> 420.4 mm, vias 2 -> 4
- net /leds+mosfets/0frame7: track 11.2 -> 236.9 mm, vias 0 -> 5
- net /leds+mosfets/0frame8: track 24.4 -> 240.8 mm, vias 0 -> 6
- net /leds+mosfets/0frame1: track 0.00 -> 201.7 mm, vias 0 -> 2
- net /leds+mosfets/0frame16: track 0.00 -> 176.7 mm, vias 0 -> 4
- net /leds+mosfets/frame12: track 0.00 -> 167.4 mm, vias 0 -> 3
- net /leds+mosfets/7or8: track 469.1 -> 617.8 mm, vias 7 -> 10
- net /leds+mosfets/0frame10: track 39.7 -> 145.3 mm, vias 2 -> 4
- net /leds+mosfets/15or16: track 0.00 -> 103.4 mm, vias 0 -> 2
- net /leds+mosfets/0frame13: track 0.00 -> 99.7 mm, vias 0 -> 3
- net /leds+mosfets/frame16: track 0.00 -> 87.1 mm, vias 0 -> 2
- net /leds+mosfets/0frame12: track 0.00 -> 78.2 mm, vias 0 -> 2
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- added copper zone on In2.Cu, net +3.3V
- removed copper zone on In2.Cu, net +2V2
