File: grad-cap-pcb/leds+mosfets.kicad_sch (KiCad schematic)
At the start: 146 parts

Commit message: addd more
switched from npn to pnp to make the LEDs connect to the ground plane - easier routing.
added labels and or gates so the mosfets wouldnt trigger each other
Parts:
- removed D19, D46: LED, LED_SMD:LED_0603_1608Metric, symbol Device:LED
- added Q1, Q10, Q11, Q12, Q13, Q14, Q15, Q16, Q2, Q3, Q4, Q5, Q6, Q7, Q8, Q9: NPN, General Library:PN2907A, symbol Simulation_SPICE:NPN
- added T1, T2: PHPT610035PKX, LFPAK56D_SOT1205_NEX, symbol PHPT610035PKX_TRANS-2PNP-100V-3A:PHPT610035PKX
- added U1, U2, U8: SN74AHCT32DBR, GRAD-CAP:SN74AHCT32DBR_2-INPUT-QUAD-OR, symbol SN74AHCT32DBR_2-INPUT-QUAD-OR:SN74AHCT32DBR
- added U3: CD4072BM96, GRAD-CAP:CD4072BM96_4-INPUT-OR, symbol CD4072BM96_4-INPUT-OR:CD4072BM96
- added U6: CD4075BM96, GRAD-CAP:CD4075BM96-3IN-TRIO-OR, symbol CD4075BM96-3IN-TRIO-OR:CD4075BM96
Connections:
- net at D130.1 (K): now also D127.1 (K), D128.1 (K), D129.1 (K), D131.1 (K), D132.1 (K)
- net 5or6: now reaches D130.2 (A)
- net 5or6: now also D131.2 (A), D132.2 (A), D135.2 (A), D136.2 (A), D137.2 (A), D138.2 (A), U8.6 (2Y)
- net frame5: now reaches D127.2 (A)
- net frame5: now also D14.2 (A), D17.2 (A), Q4.1 (C), U3.2 (A), U8.12 (4A), U8.4 (2A)
- net at D7.1 (K): now also D10.1 (K), D11.1 (K), D12.1 (K), D8.1 (K), D9.1 (K)
- net frame4: now reaches D7.2 (A)
- net frame4: now also D10.2 (A), D11.2 (A), D114.2 (A), D116.2 (A), D117.2 (A), D118.2 (A), D12.2 (A), D120.2 (A), D123.2 (A), D129.2 (A), D18.2 (A), D8.2 (A), D9.2 (A), Q3.1 (C), U8.13 (4B), U8.2 (1B)
- net at D136.1 (K): now also D133.1 (K), D134.1 (K), D135.1 (K), D137.1 (K), D138.1 (K)
- net at D115.1 (K): now also D116.1 (K), D117.1 (K), D118.1 (K), D119.1 (K), D120.1 (K)
- net frame3: now reaches D115.2 (A)
- net frame3: now also D111.2 (A), D112.2 (A), D119.2 (A), D5.2 (A), D6.2 (A), Q2.1 (C), U8.1 (1A)
- net at D124.1 (K): now also D121.1 (K), D122.1 (K), D123.1 (K), D125.1 (K), D126.1 (K)
- net 4or5: now reaches D124.2 (A)
- net 4or5: now also D121.2 (A), D122.2 (A), D125.2 (A), D126.2 (A), D128.2 (A), D13.2 (A), D133.2 (A), D15.2 (A), D16.2 (A), U8.11 (4Y)
- net at D2.1 (K): now also D1.1 (K), D3.1 (K), D4.1 (K), D5.1 (K), D6.1 (K)
- net frame1: now reaches D2.2 (A)
- net frame1: now also D1.2 (A), D108.2 (A), D109.2 (A), Q16.1 (C), U6.11 (I)
- net at D49.1 (K): now also D45.1 (K), D47.1 (K), D48.1 (K), D50.1 (K), D51.1 (K)
- net 7or8: now reaches D49.2 (A)
- net 7or8: now also D146.2 (A), D30.2 (A), D31.2 (A), D33.2 (A), D36.2 (A), D37.2 (A), D39.2 (A), D48.2 (A), D53.2 (A), D56.2 (A), U2.3 (1Y)
- net at D74.1 (K): now also D73.1 (K), D75.1 (K), D76.1 (K), D77.1 (K), D78.1 (K)
- net frame13: now reaches D74.2 (A)
- net frame13: now also D69.2 (A), D70.2 (A), D71.2 (A), D76.2 (A), D78.2 (A), D79.2 (A), D81.2 (A), D93.2 (A), Q12.1 (C), U1.1 (1A), U8.9 (3A)
- net at D94.1 (K): now also D91.1 (K), D92.1 (K), D93.1 (K), D95.1 (K), D96.1 (K)
- net 14or15: now reaches D94.2 (A)
- net 14or15: now also D104.2 (A), D85.2 (A), D87.2 (A), D90.2 (A), D96.2 (A), U1.6 (2Y)
- net at D20.1 (K): now also D22.1 (K), D23.1 (K), D24.1 (K), D25.1 (K), D26.1 (K)
- net 6or7: now reaches D20.2 (A)
- net 6or7: now also D139.2 (A), D140.2 (A), D141.2 (A), D145.2 (A), D22.2 (A), D27.2 (A), D28.2 (A), D32.2 (A), D34.2 (A), U2.6 (2Y)
- net at D15.1 (K): now also D13.1 (K), D14.1 (K), D16.1 (K), D17.1 (K), D18.1 (K)
- net at D37.1 (K): now also D33.1 (K), D34.1 (K), D35.1 (K), D36.1 (K), D38.1 (K)
- net at D86.1 (K): now also D85.1 (K), D87.1 (K), D88.1 (K), D89.1 (K), D90.1 (K)
- net 13or14: now reaches D86.2 (A)
- net 13or14: now also D102.2 (A), D77.2 (A), D84.2 (A), U1.3 (1Y)
- net at D54.1 (K): now also D52.1 (K), D53.1 (K)
- net frame9: now reaches D54.2 (A)
- net frame9: now also D47.2 (A), D58.2 (A), D59.2 (A), Q8.1 (C), U1.10 (3B), U2.12 (4A), U6.2 (B), U6.5 (D)
- net at D65.1 (K): now also D61.1 (K), D62.1 (K), D63.1 (K), D64.1 (K), D66.1 (K)
- net frame12: now reaches D65.2 (A)
- net frame12: now also D63.2 (A), D64.2 (A), D66.2 (A), D67.2 (A), D73.2 (A), Q11.1 (C), U8.10 (3B)
- net at D141.1 (K): now also D139.1 (K), D140.1 (K), D142.1 (K), D143.1 (K), D144.1 (K)
- net at D99.1 (K): now also D100.1 (K), D101.1 (K), D102.1 (K), D97.1 (K), D98.1 (K)
- net 15or16: now reaches D99.2 (A)
- net 15or16: now also D106.2 (A), U1.11 (4Y)
- net at D70.1 (K): now also D67.1 (K), D68.1 (K), D69.1 (K), D71.1 (K), D72.1 (K)
- net frame6: now reaches D35.2 (A)
- net frame6: now also D134.2 (A), D23.2 (A), D24.2 (A), D25.2 (A), D26.2 (A), Q5.1 (C), U2.4 (2A), U3.12 (H), U3.3 (B), U8.5 (2B)
- net at D56.1 (K): now also D55.1 (K), D57.1 (K), D58.1 (K), D59.1 (K), D60.1 (K)
- net at D110.1 (K): now also D109.1 (K), D111.1 (K), D112.1 (K), D113.1 (K), D114.1 (K)
- net frame2: now reaches D110.2 (A)
- net frame2: now also D3.2 (A), D4.2 (A), Q1.1 (C)
- net frame7: now reaches D38.2 (A)
- net frame7: now also D147.2 (A), D29.2 (A), D45.2 (A), D55.2 (A), Q6.1 (C), U2.1 (1A), U2.5 (2B), U3.11 (G), U3.4 (C), U6.3 (F)
- net at D106.1 (K): now also D103.1 (K), D104.1 (K), D105.1 (K), D107.1 (K), D108.1 (K)
- net 5or6or7or8: now reaches D142.2 (A)
- net 5or6or7or8: now also U3.1 (J)
- net 6or7or8: now reaches D144.2 (A)
- net 6or7or8: now also D143.2 (A), U3.13 (K)
- net at D31.1 (K): now also D27.1 (K), D28.1 (K), D29.1 (K), D30.1 (K), D32.1 (K)
- net frame8: now reaches D57.2 (A)
- net frame8: now also Q7.1 (C), U2.13 (4B), U2.2 (1B), U3.10 (F), U3.5 (D), U6.4 (E), U6.8 (A)
- net frame14: now reaches D75.2 (A)
- net frame14: now also D100.2 (A), D103.2 (A), D80.2 (A), D82.2 (A), D88.2 (A), D89.2 (A), D91.2 (A), D97.2 (A), Q13.1 (C), U1.2 (1B), U1.4 (2A)
- net 12or13: now reaches D72.2 (A)
- net 12or13: now also D68.2 (A), D83.2 (A), U8.8 (3Y)
- net 7or8or9: now reaches D52.2 (A)
- net 7or8or9: now also D43.2 (A), U6.6 (K)
- net at D84.1 (K): now also D79.1 (K), D80.1 (K), D81.1 (K), D82.1 (K), D83.1 (K)
- net frame16: now reaches D95.2 (A)
- net frame16: now also D107.2 (A), Q15.1 (C), U1.12 (4A), U6.12 (H)
- net 8or9or10: now reaches D51.2 (A)
- net 8or9or10: now also U6.9 (J)
- net 10or11: now reaches D60.2 (A)
- net 10or11: now also U2.8 (3Y)
- net frame15: now reaches D101.2 (A)
- net frame15: now also D105.2 (A), D92.2 (A), D98.2 (A), Q14.1 (C), U1.13 (4B), U1.5 (2B)
- net 9or10: now reaches D50.2 (A)
- net 9or10: now also U1.8 (3Y)
- net at D147.1 (K): now also D145.1 (K), D146.1 (K)
- net at D39.1 (K): now also D40.1 (K), D41.1 (K), D42.1 (K), D43.1 (K), D44.1 (K)
- net frame11: now reaches D61.2 (A)
- net frame11: now also D62.2 (A), Q10.1 (C), U2.9 (3A)
- net 8or9: now reaches D42.2 (A)
- net 8or9: now also D40.2 (A), D41.2 (A), D44.2 (A), U2.11 (4Y)
- net 3or4: now reaches D113.2 (A)
- net 3or4: now also U8.3 (1Y)
- new net +3.3V: U1.14 (VCC), U2.14 (VCC), U3.14 (VDD), U6.14 (VDD), U8.14 (VCC)
- new net 0: Q16.2 (B)
- new net 1: Q1.2 (B)
- new net 10: Q10.2 (B)
- new net 11: Q11.2 (B)
- new net 12: Q12.2 (B)
- new net 13: Q13.2 (B)
- new net 14: Q14.2 (B)
- new net 15: Q15.2 (B)
- new net 16or1: U6.10 (L)
- new net 2: Q2.2 (B)
- new net 3: Q3.2 (B)
- new net 4: Q4.2 (B)
- new net 5: Q5.2 (B)
- new net 6: Q6.2 (B)
- new net 7: Q7.2 (B)
- new net 8: Q8.2 (B)
- new net 9: Q9.2 (B)
- new net GND: U1.7 (GND), U2.7 (GND), U3.7 (VSS), U3.9 (E), U6.13 (G), U8.7 (GND)
- new net frame10: Q9.1 (C), U1.9 (3A), U2.10 (3B), U6.1 (C)
Other:
- note added: "CENTER FIREWORK"
- note added: "LEFT FIREWORK"
- note added: "OR GATES"

Commit message: added many things
added: mux
counter
signal gen - still needs r1 and r2 values
power management
kicad symbol library - footprints not assigned
Parts:
- removed Q1, Q10, Q11, Q12, Q13, Q14, Q15, Q16, Q2, Q3, Q4, Q5, Q6, Q7, Q8, Q9: NPN, General Library:PN2907A, symbol Simulation_SPICE:NPN
- added T3, T4, T5, T6, T7, T8: PHPT610035PKX, GRAD-CAP:PHPT610035PKX_TRANS-2PNP-100V-3A, symbol PHPT610035PKX_TRANS-2PNP-100V-3A:PHPT610035PKX
- T1, T2: footprint LFPAK56D_SOT1205_NEX -> GRAD-CAP:PHPT610035PKX_TRANS-2PNP-100V-3A
Connections:
- net 0: now also T1.2 (BASE)
- net 1: now also T1.4 (BASE)
- net 10: now also T6.2 (BASE)
- net 10or11: now also D60.1 (K); no longer D60.2 (A)
- net 11: now also T6.4 (BASE)
- net 12: now also T7.2 (BASE)
- net 12or13: now also D68.1 (K), D72.1 (K), D83.1 (K); no longer D68.2 (A), D72.2 (A), D83.2 (A)
- net 13: now also T7.4 (BASE)
- net 13or14: now also D102.1 (K), D77.1 (K), D84.1 (K), D86.1 (K); no longer D102.2 (A), D77.2 (A), D84.2 (A), D86.2 (A)
- net 14: now also T8.2 (BASE)
- net 14or15: now also D104.1 (K), D85.1 (K), D87.1 (K), D90.1 (K), D94.1 (K), D96.1 (K); no longer D104.2 (A), D85.2 (A), D87.2 (A), D90.2 (A), D94.2 (A), D96.2 (A)
- net 15: now also T8.4 (BASE)
- net 15or16: now also D106.1 (K), D99.1 (K); no longer D106.2 (A), D99.2 (A)
- net 2: now also T2.2 (BASE)
- net 3: now also T2.4 (BASE)
- net 3or4: now also D113.1 (K); no longer D113.2 (A)
- net 4: now also T3.2 (BASE)
- net 4or5: now also D121.1 (K), D122.1 (K), D124.1 (K), D125.1 (K), D126.1 (K), D128.1 (K), D13.1 (K), D133.1 (K), D15.1 (K), D16.1 (K); no longer D121.2 (A), D122.2 (A), D124.2 (A), D125.2 (A), D126.2 (A), D128.2 (A), D13.2 (A), D133.2 (A), D15.2 (A), D16.2 (A)
- net 5: now also T3.4 (BASE)
- net 5or6: now also D130.1 (K), D131.1 (K), D132.1 (K), D135.1 (K), D136.1 (K), D137.1 (K), D138.1 (K); no longer D130.2 (A), D131.2 (A), D132.2 (A), D135.2 (A), D136.2 (A), D137.2 (A), D138.2 (A)
- net 5or6or7or8: now also D142.1 (K); no longer D142.2 (A)
- net 6: now also T4.2 (BASE)
- net 6or7: now also D139.1 (K), D140.1 (K), D141.1 (K), D145.1 (K), D20.1 (K), D22.1 (K), D27.1 (K), D28.1 (K), D32.1 (K), D34.1 (K); no longer D139.2 (A), D140.2 (A), D141.2 (A), D145.2 (A), D20.2 (A), D22.2 (A), D27.2 (A), D28.2 (A), D32.2 (A), D34.2 (A)
- net 6or7or8: now also D143.1 (K), D144.1 (K); no longer D143.2 (A), D144.2 (A)
- net 7: now also T4.4 (BASE)
- net 7or8: now also D146.1 (K), D30.1 (K), D31.1 (K), D33.1 (K), D36.1 (K), D37.1 (K), D39.1 (K), D48.1 (K), D49.1 (K), D53.1 (K), D56.1 (K); no longer D146.2 (A), D30.2 (A), D31.2 (A), D33.2 (A), D36.2 (A), D37.2 (A), D39.2 (A), D48.2 (A), D49.2 (A), D53.2 (A), D56.2 (A)
- net 7or8or9: now also D43.1 (K), D52.1 (K); no longer D43.2 (A), D52.2 (A)
- net 8: now also T5.2 (BASE)
- net 8or9: now also D40.1 (K), D41.1 (K), D42.1 (K), D44.1 (K); no longer D40.2 (A), D41.2 (A), D42.2 (A), D44.2 (A)
- net 8or9or10: now also D51.1 (K); no longer D51.2 (A)
- net 9: now also T5.4 (BASE)
- net 9or10: now also D50.1 (K); no longer D50.2 (A)
- net frame1: now also D1.1 (K), D108.1 (K), D109.1 (K), D2.1 (K), T1.7 (COLLECTOR), T1.8 (COLLECTOR); no longer D1.2 (A), D108.2 (A), D109.2 (A), D2.2 (A)
- net frame10: now also T5.5 (COLLECTOR), T5.6 (COLLECTOR)
- net frame11: now also D61.1 (K), D62.1 (K), T6.7 (COLLECTOR), T6.8 (COLLECTOR); no longer D61.2 (A), D62.2 (A)
- net frame12: now also D63.1 (K), D64.1 (K), D65.1 (K), D66.1 (K), D67.1 (K), D73.1 (K), T6.5 (COLLECTOR), T6.6 (COLLECTOR); no longer D63.2 (A), D64.2 (A), D65.2 (A), D66.2 (A), D67.2 (A), D73.2 (A)
- net frame13: now also D69.1 (K), D70.1 (K), D71.1 (K), D74.1 (K), D76.1 (K), D78.1 (K), D79.1 (K), D81.1 (K), D93.1 (K), T7.7 (COLLECTOR), T7.8 (COLLECTOR); no longer D69.2 (A), D70.2 (A), D71.2 (A), D74.2 (A), D76.2 (A), D78.2 (A), D79.2 (A), D81.2 (A), D93.2 (A)
- net frame14: now also D100.1 (K), D103.1 (K), D75.1 (K), D80.1 (K), D82.1 (K), D88.1 (K), D89.1 (K), D91.1 (K), D97.1 (K), T7.5 (COLLECTOR), T7.6 (COLLECTOR); no longer D100.2 (A), D103.2 (A), D75.2 (A), D80.2 (A), D82.2 (A), D88.2 (A), D89.2 (A), D91.2 (A), D97.2 (A)
- net frame15: now also D101.1 (K), D105.1 (K), D92.1 (K), D98.1 (K), T8.7 (COLLECTOR), T8.8 (COLLECTOR); no longer D101.2 (A), D105.2 (A), D92.2 (A), D98.2 (A)
- net frame16: now also D107.1 (K), D95.1 (K), T8.5 (COLLECTOR), T8.6 (COLLECTOR); no longer D107.2 (A), D95.2 (A)
- net frame2: now also D110.1 (K), D3.1 (K), D4.1 (K), T1.5 (COLLECTOR), T1.6 (COLLECTOR); no longer D110.2 (A), D3.2 (A), D4.2 (A)
- net frame3: now also D111.1 (K), D112.1 (K), D115.1 (K), D119.1 (K), D5.1 (K), D6.1 (K), T2.7 (COLLECTOR), T2.8 (COLLECTOR); no longer D111.2 (A), D112.2 (A), D115.2 (A), D119.2 (A), D5.2 (A), D6.2 (A)
- net frame4: now also D10.1 (K), D11.1 (K), D114.1 (K), D116.1 (K), D117.1 (K), D118.1 (K), D12.1 (K), D120.1 (K), D123.1 (K), D129.1 (K), D18.1 (K), D7.1 (K), D8.1 (K), D9.1 (K), T2.5 (COLLECTOR), T2.6 (COLLECTOR); no longer D10.2 (A), D11.2 (A), D114.2 (A), D116.2 (A), D117.2 (A), D118.2 (A), D12.2 (A), D120.2 (A), D123.2 (A), D129.2 (A), D18.2 (A), D7.2 (A), D8.2 (A), D9.2 (A)
- net frame5: now also D127.1 (K), D14.1 (K), D17.1 (K), T3.7 (COLLECTOR), T3.8 (COLLECTOR); no longer D127.2 (A), D14.2 (A), D17.2 (A)
- net frame6: now also D134.1 (K), D23.1 (K), D24.1 (K), D25.1 (K), D26.1 (K), D35.1 (K), T3.5 (COLLECTOR), T3.6 (COLLECTOR); no longer D134.2 (A), D23.2 (A), D24.2 (A), D25.2 (A), D26.2 (A), D35.2 (A)
- net frame7: now also D147.1 (K), D29.1 (K), D38.1 (K), D45.1 (K), D55.1 (K), T4.7 (COLLECTOR), T4.8 (COLLECTOR); no longer D147.2 (A), D29.2 (A), D38.2 (A), D45.2 (A), D55.2 (A)
- net frame8: now also D57.1 (K), T4.5 (COLLECTOR), T4.6 (COLLECTOR); no longer D57.2 (A)
- net frame9: now also D47.1 (K), D54.1 (K), D58.1 (K), D59.1 (K), T5.7 (COLLECTOR), T5.8 (COLLECTOR); no longer D47.2 (A), D54.2 (A), D58.2 (A), D59.2 (A)
- net +2V2: now reaches T1.1 (EMITTER)
- net +2V2: now also T1.3 (EMITTER), T2.1 (EMITTER), T2.3 (EMITTER), T3.1 (EMITTER), T3.3 (EMITTER), T4.1 (EMITTER), T4.3 (EMITTER), T5.1 (EMITTER), T5.3 (EMITTER), T6.1 (EMITTER), T6.3 (EMITTER), T7.1 (EMITTER), T7.3 (EMITTER), T8.1 (EMITTER), T8.3 (EMITTER)
- new net: D10.2 (A), D11.2 (A), D12.2 (A), D7.2 (A), D8.2 (A), D9.2 (A)
- new net: D61.2 (A), D62.2 (A), D63.2 (A), D64.2 (A), D65.2 (A), D66.2 (A)
- new net: D45.2 (A), D47.2 (A), D48.2 (A), D49.2 (A), D50.2 (A), D51.2 (A)
- new net: D139.2 (A), D140.2 (A), D141.2 (A), D142.2 (A), D143.2 (A), D144.2 (A)
- new net: D55.2 (A), D56.2 (A), D57.2 (A), D58.2 (A), D59.2 (A), D60.2 (A)
- new net: D13.2 (A), D14.2 (A), D15.2 (A), D16.2 (A), D17.2 (A), D18.2 (A)
- new net: D73.2 (A), D74.2 (A), D75.2 (A), D76.2 (A), D77.2 (A), D78.2 (A)
- new net: D100.2 (A), D101.2 (A), D102.2 (A), D97.2 (A), D98.2 (A), D99.2 (A)
- new net: D39.2 (A), D40.2 (A), D41.2 (A), D42.2 (A), D43.2 (A), D44.2 (A)
- new net: D27.2 (A), D28.2 (A), D29.2 (A), D30.2 (A), D31.2 (A), D32.2 (A)
- new net: D85.2 (A), D86.2 (A), D87.2 (A), D88.2 (A), D89.2 (A), D90.2 (A)
- new net: D133.2 (A), D134.2 (A), D135.2 (A), D136.2 (A), D137.2 (A), D138.2 (A)
- new net: D33.2 (A), D34.2 (A), D35.2 (A), D36.2 (A), D37.2 (A), D38.2 (A)
- new net: D127.2 (A), D128.2 (A), D129.2 (A), D130.2 (A), D131.2 (A), D132.2 (A)
- new net: D67.2 (A), D68.2 (A), D69.2 (A), D70.2 (A), D71.2 (A), D72.2 (A)
- new net: D20.2 (A), D22.2 (A), D23.2 (A), D24.2 (A), D25.2 (A), D26.2 (A)
- new net: D79.2 (A), D80.2 (A), D81.2 (A), D82.2 (A), D83.2 (A), D84.2 (A)
- new net: D145.2 (A), D146.2 (A), D147.2 (A)
- new net: D52.2 (A), D53.2 (A), D54.2 (A)
- new net: D121.2 (A), D122.2 (A), D123.2 (A), D124.2 (A), D125.2 (A), D126.2 (A)
- new net: D109.2 (A), D110.2 (A), D111.2 (A), D112.2 (A), D113.2 (A), D114.2 (A)
- new net: D1.2 (A), D2.2 (A), D3.2 (A), D4.2 (A), D5.2 (A), D6.2 (A)
- new net: D115.2 (A), D116.2 (A), D117.2 (A), D118.2 (A), D119.2 (A), D120.2 (A)
- new net: D91.2 (A), D92.2 (A), D93.2 (A), D94.2 (A), D95.2 (A), D96.2 (A)
- new net: D103.2 (A), D104.2 (A), D105.2 (A), D106.2 (A), D107.2 (A), D108.2 (A)
Other:
- note added: "MOSFETS"
- moved on the sheet: D1, D2, D3, D4, D5, D6, T1, T2, U1, U2, U3, U6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

Commit message: edited layout
Parts:
- renumbered U3 to U1, U6 to U2, U8 to U3, U1 to U6, U2 to U8
Connections:
- net 0: now also T1.4 (BASE); no longer T1.2 (BASE)
- net 1: now also T1.2 (BASE); no longer T1.4 (BASE)
- net 10: now also T6.4 (BASE); no longer T6.2 (BASE)
- net 11: now also T6.2 (BASE); no longer T6.4 (BASE)
- net 12: now also T7.4 (BASE); no longer T7.2 (BASE)
- net 12or13: now also D68.2 (A), D72.2 (A), D83.2 (A); no longer D68.1 (K), D72.1 (K), D83.1 (K)
- net 13: now also T7.2 (BASE); no longer T7.4 (BASE)
- net 13or14: now also D102.2 (A), D77.2 (A), D84.2 (A), D86.2 (A); no longer D102.1 (K), D77.1 (K), D84.1 (K), D86.1 (K)
- net 14: now also T8.4 (BASE); no longer T8.2 (BASE)
- net 14or15: now also D85.2 (A), D87.2 (A), D90.2 (A), D94.2 (A), D96.2 (A); no longer D104.1 (K), D85.1 (K), D87.1 (K), D90.1 (K), D94.1 (K), D96.1 (K)
- net 15: now also T8.2 (BASE); no longer T8.4 (BASE)
- net 15or16: now also D101.2 (A), D106.2 (A), D95.2 (A), D99.2 (A); no longer D106.1 (K), D99.1 (K)
- net 2: now also T2.4 (BASE); no longer T2.2 (BASE)
- net 3: now also T2.2 (BASE); no longer T2.4 (BASE)
- net 3or4: now also D113.2 (A); no longer D113.1 (K)
- net 4: now also T3.4 (BASE); no longer T3.2 (BASE)
- net 4or5: now also D121.2 (A), D122.2 (A), D124.2 (A), D125.2 (A), D126.2 (A), D128.2 (A), D13.2 (A), D133.2 (A), D15.2 (A), D16.2 (A); no longer D121.1 (K), D122.1 (K), D124.1 (K), D125.1 (K), D126.1 (K), D128.1 (K), D13.1 (K), D133.1 (K), D15.1 (K), D16.1 (K)
- net 5: now also T3.2 (BASE); no longer T3.4 (BASE)
- net 5or6: now also D130.2 (A), D131.2 (A), D132.2 (A), D135.2 (A), D136.2 (A), D137.2 (A), D138.2 (A); no longer D130.1 (K), D131.1 (K), D132.1 (K), D135.1 (K), D136.1 (K), D137.1 (K), D138.1 (K)
- net 5or6or7or8: now also D142.2 (A); no longer D142.1 (K)
- net 6: now also T4.4 (BASE); no longer T4.2 (BASE)
- net 6or7: now also D139.2 (A), D140.2 (A), D141.2 (A), D145.2 (A), D20.2 (A), D22.2 (A), D27.2 (A), D28.2 (A), D32.2 (A), D34.2 (A); no longer D139.1 (K), D140.1 (K), D141.1 (K), D145.1 (K), D20.1 (K), D22.1 (K), D27.1 (K), D28.1 (K), D32.1 (K), D34.1 (K)
- net 6or7or8: now also D143.2 (A), D144.2 (A); no longer D143.1 (K), D144.1 (K)
- net 7: now also T4.2 (BASE); no longer T4.4 (BASE)
- net 7or8: now also D146.2 (A), D30.2 (A), D31.2 (A), D33.2 (A), D36.2 (A), D37.2 (A), D39.2 (A), D48.2 (A), D49.2 (A), D53.2 (A), D56.2 (A); no longer D146.1 (K), D30.1 (K), D31.1 (K), D33.1 (K), D36.1 (K), D37.1 (K), D39.1 (K), D48.1 (K), D49.1 (K), D53.1 (K), D56.1 (K)
- net 7or8or9: now also D43.2 (A), D52.2 (A); no longer D43.1 (K), D52.1 (K)
- net 8: now also T5.4 (BASE); no longer T5.2 (BASE)
- net 8or9: now also D40.2 (A), D41.2 (A), D42.2 (A), D44.2 (A); no longer D40.1 (K), D41.1 (K), D42.1 (K), D44.1 (K)
- net 8or9or10: now also D51.2 (A); no longer D51.1 (K)
- net 9: now also T5.2 (BASE); no longer T5.4 (BASE)
- net 9or10: now also D50.2 (A); no longer D50.1 (K)
- net GND: now also D1.1 (K), D10.1 (K), D100.1 (K), D101.1 (K), D102.1 (K), D103.1 (K), D104.1 (K), D105.1 (K), D106.1 (K), D107.1 (K), D108.1 (K), D109.1 (K), D11.1 (K), D110.1 (K), D111.1 (K), D112.1 (K), D113.1 (K), D114.1 (K), D115.1 (K), D116.1 (K), D117.1 (K), D118.1 (K), D119.1 (K), D12.1 (K), D120.1 (K), D121.1 (K), D122.1 (K), D123.1 (K), D124.1 (K), D125.1 (K), D126.1 (K), D127.1 (K), D128.1 (K), D129.1 (K), D13.1 (K), D130.1 (K), D131.1 (K), D132.1 (K), D133.1 (K), D134.1 (K), D135.1 (K), D136.1 (K), D137.1 (K), D138.1 (K), D139.1 (K), D14.1 (K), D140.1 (K), D141.1 (K), D142.1 (K), D143.1 (K), D144.1 (K), D145.1 (K), D146.1 (K), D147.1 (K), D15.1 (K), D16.1 (K), D17.1 (K), D18.1 (K), D2.1 (K), D20.1 (K), D22.1 (K), D23.1 (K), D24.1 (K), D25.1 (K), D26.1 (K), D27.1 (K), D28.1 (K), D29.1 (K), D3.1 (K), D30.1 (K), D31.1 (K), D32.1 (K), D33.1 (K), D34.1 (K), D35.1 (K), D36.1 (K), D37.1 (K), D38.1 (K), D39.1 (K), D4.1 (K), D40.1 (K), D41.1 (K), D42.1 (K), D43.1 (K), D44.1 (K), D45.1 (K), D47.1 (K), D48.1 (K), D49.1 (K), D5.1 (K), D50.1 (K), D51.1 (K), D52.1 (K), D53.1 (K), D54.1 (K), D55.1 (K), D56.1 (K), D57.1 (K), D58.1 (K), D59.1 (K), D6.1 (K), D60.1 (K), D61.1 (K), D62.1 (K), D63.1 (K), D64.1 (K), D65.1 (K), D66.1 (K), D67.1 (K), D68.1 (K), D69.1 (K), D7.1 (K), D70.1 (K), D71.1 (K), D72.1 (K), D73.1 (K), D74.1 (K), D75.1 (K), D76.1 (K), D77.1 (K), D78.1 (K), D79.1 (K), D8.1 (K), D80.1 (K), D81.1 (K), D82.1 (K), D83.1 (K), D84.1 (K), D85.1 (K), D86.1 (K), D87.1 (K), D88.1 (K), D89.1 (K), D9.1 (K), D90.1 (K), D91.1 (K), D92.1 (K), D93.1 (K), D94.1 (K), D95.1 (K), D96.1 (K), D97.1 (K), D98.1 (K), D99.1 (K)
- net frame1: now also D1.2 (A), D108.2 (A), D109.2 (A), D2.2 (A), T1.5 (COLLECTOR), T1.6 (COLLECTOR); no longer D1.1 (K), D108.1 (K), D109.1 (K), D2.1 (K), T1.7 (COLLECTOR), T1.8 (COLLECTOR)
- net frame10: now also D60.2 (A), T5.7 (COLLECTOR), T5.8 (COLLECTOR); no longer T5.5 (COLLECTOR), T5.6 (COLLECTOR), U8.10 (3B)
- net frame11: now also D61.2 (A), D62.2 (A), T6.5 (COLLECTOR), T6.6 (COLLECTOR); no longer D61.1 (K), D62.1 (K), T6.7 (COLLECTOR), T6.8 (COLLECTOR), U8.9 (3A)
- net frame12: now also D63.2 (A), D64.2 (A), D65.2 (A), D66.2 (A), D67.2 (A), D73.2 (A), T6.7 (COLLECTOR), T6.8 (COLLECTOR); no longer D63.1 (K), D64.1 (K), D65.1 (K), D66.1 (K), D67.1 (K), D73.1 (K), T6.5 (COLLECTOR), T6.6 (COLLECTOR)
- net frame13: now also D69.2 (A), D70.2 (A), D71.2 (A), D74.2 (A), D76.2 (A), D78.2 (A), D79.2 (A), D81.2 (A), D93.2 (A), T7.5 (COLLECTOR), T7.6 (COLLECTOR); no longer D69.1 (K), D70.1 (K), D71.1 (K), D74.1 (K), D76.1 (K), D78.1 (K), D79.1 (K), D81.1 (K), D93.1 (K), T7.7 (COLLECTOR), T7.8 (COLLECTOR)
- net frame14: now also D100.2 (A), D75.2 (A), D80.2 (A), D82.2 (A), D88.2 (A), D89.2 (A), D91.2 (A), D97.2 (A), T7.7 (COLLECTOR), T7.8 (COLLECTOR); no longer D100.1 (K), D103.1 (K), D75.1 (K), D80.1 (K), D82.1 (K), D88.1 (K), D89.1 (K), D91.1 (K), D97.1 (K), T7.5 (COLLECTOR), T7.6 (COLLECTOR)
- net frame15: now also D104.2 (A), D105.2 (A), D92.2 (A), D98.2 (A), T8.5 (COLLECTOR), T8.6 (COLLECTOR); no longer D101.1 (K), D105.1 (K), D92.1 (K), D98.1 (K), T8.7 (COLLECTOR), T8.8 (COLLECTOR)
- net frame16: now also D107.2 (A), T8.7 (COLLECTOR), T8.8 (COLLECTOR); no longer D107.1 (K), D95.1 (K), T8.5 (COLLECTOR), T8.6 (COLLECTOR)
- net frame2: now also D110.2 (A), D3.2 (A), D4.2 (A), T1.7 (COLLECTOR), T1.8 (COLLECTOR); no longer D110.1 (K), D3.1 (K), D4.1 (K), T1.5 (COLLECTOR), T1.6 (COLLECTOR)
- net frame3: now also D111.2 (A), D112.2 (A), D115.2 (A), D119.2 (A), D5.2 (A), D6.2 (A), T2.5 (COLLECTOR), T2.6 (COLLECTOR); no longer D111.1 (K), D112.1 (K), D115.1 (K), D119.1 (K), D5.1 (K), D6.1 (K), T2.7 (COLLECTOR), T2.8 (COLLECTOR)
- net frame4: now also D10.2 (A), D11.2 (A), D114.2 (A), D116.2 (A), D117.2 (A), D118.2 (A), D12.2 (A), D120.2 (A), D123.2 (A), D129.2 (A), D18.2 (A), D7.2 (A), D8.2 (A), D9.2 (A), T2.7 (COLLECTOR), T2.8 (COLLECTOR); no longer D10.1 (K), D11.1 (K), D114.1 (K), D116.1 (K), D117.1 (K), D118.1 (K), D12.1 (K), D120.1 (K), D123.1 (K), D129.1 (K), D18.1 (K), D7.1 (K), D8.1 (K), D9.1 (K), T2.5 (COLLECTOR), T2.6 (COLLECTOR)
- net frame5: now also D127.2 (A), D14.2 (A), D17.2 (A), T3.5 (COLLECTOR), T3.6 (COLLECTOR); no longer D127.1 (K), D14.1 (K), D17.1 (K), T3.7 (COLLECTOR), T3.8 (COLLECTOR)
- net frame6: now also D134.2 (A), D23.2 (A), D24.2 (A), D25.2 (A), D26.2 (A), D35.2 (A), T3.7 (COLLECTOR), T3.8 (COLLECTOR); no longer D134.1 (K), D23.1 (K), D24.1 (K), D25.1 (K), D26.1 (K), D35.1 (K), T3.5 (COLLECTOR), T3.6 (COLLECTOR)
- net frame7: now also D147.2 (A), D29.2 (A), D38.2 (A), D45.2 (A), D55.2 (A), T4.5 (COLLECTOR), T4.6 (COLLECTOR); no longer D147.1 (K), D29.1 (K), D38.1 (K), D45.1 (K), D55.1 (K), T4.7 (COLLECTOR), T4.8 (COLLECTOR)
- net frame8: now also D57.2 (A), T4.7 (COLLECTOR), T4.8 (COLLECTOR); no longer D57.1 (K), T4.5 (COLLECTOR), T4.6 (COLLECTOR)
- net frame9: now also D47.2 (A), D54.2 (A), D58.2 (A), D59.2 (A), T5.5 (COLLECTOR), T5.6 (COLLECTOR); no longer D47.1 (K), D54.1 (K), D58.1 (K), D59.1 (K), T5.7 (COLLECTOR), T5.8 (COLLECTOR)
- net 10or11: no longer names the net of U8.8 (3Y)
- net 10or11: no longer D60.1 (K)
- now unconnected: D103.2 (A)
- no-connect marks 0 -> 3
Other:
- note added: "2-INPUT-QUAD-OR"
- note added: "3IN-TRIO-OR"
- note added: "4-INPUT-OR"
- moved on the sheet: D1, D2, D3, D4, D5, D6

Commit message: routed traces, added resistors
Parts:
- added R11, R12, R13, R14, R15, R16, R17, R18, R19, R2, R20, R21, R22, R23, R24, R25, R26, R27, R28, R29, R3, R30, R31, R32, R33, R34, R35, R36, R37, R38, R39, R40: R_Small_US, Resistor_SMD:R_0805_2012Metric_Pad1.20x1.40mm_HandSolder, symbol Device:R_Small_US
Connections:
- net 12or13: now also R33.1; no longer U3.8 (3Y)
- net 13or14: now also R34.1; no longer U6.3 (1Y)
- net 14or15: now also R35.1; no longer U6.6 (2Y)
- net 15or16: now also R37.1; no longer U6.11 (4Y)
- net 16or1: now also R31.1; no longer U2.10 (L)
- net 3or4: now also R25.1; no longer U3.3 (1Y)
- net 4or5: now also R30.1; no longer U3.11 (4Y)
- net 5or6: now also R27.1; no longer U3.6 (2Y)
- net 5or6or7or8: now also R26.1; no longer U1.1 (J)
- net 6or7: now also R40.1; no longer U8.6 (2Y)
- net 6or7or8: now also R29.1; no longer U1.13 (K)
- net 7or8: now also R36.1; no longer U8.3 (1Y)
- net 7or8or9: now also R28.1; no longer U2.6 (K)
- net 8or9: now also R39.1; no longer U8.11 (4Y)
- net 8or9or10: now also R32.1; no longer U2.9 (J)
- net 9or10: now also R38.1; no longer U6.8 (3Y)
- net GND: now also U2.7 (VSS)
- net frame1: now also R2.1; no longer T1.5 (COLLECTOR), T1.6 (COLLECTOR), U2.11 (I)
- net frame10: now also R18.1; no longer T5.7 (COLLECTOR), T5.8 (COLLECTOR), U2.1 (C), U6.9 (3A)
- net frame11: now also R19.1; no longer T6.5 (COLLECTOR), T6.6 (COLLECTOR)
- net frame12: now also R20.1; no longer T6.7 (COLLECTOR), T6.8 (COLLECTOR), U3.10 (3B)
- net frame13: now also R21.1; no longer T7.5 (COLLECTOR), T7.6 (COLLECTOR), U3.9 (3A), U6.1 (1A)
- net frame14: now also R22.1; no longer T7.7 (COLLECTOR), T7.8 (COLLECTOR), U6.2 (1B), U6.4 (2A)
- net frame15: now also R23.1; no longer T8.5 (COLLECTOR), T8.6 (COLLECTOR), U6.13 (4B), U6.5 (2B)
- net frame16: now also R24.1; no longer T8.7 (COLLECTOR), T8.8 (COLLECTOR), U2.12 (H), U6.12 (4A)
- net frame2: now also R3.1; no longer T1.7 (COLLECTOR), T1.8 (COLLECTOR)
- net frame3: now also R11.1; no longer T2.5 (COLLECTOR), T2.6 (COLLECTOR), U3.1 (1A)
- net frame4: now also R12.1; no longer T2.7 (COLLECTOR), T2.8 (COLLECTOR), U3.13 (4B), U3.2 (1B)
- net frame5: now also R13.1; no longer T3.5 (COLLECTOR), T3.6 (COLLECTOR), U1.2 (A), U3.12 (4A), U3.4 (2A)
- net frame6: now also R14.1; no longer T3.7 (COLLECTOR), T3.8 (COLLECTOR), U1.12 (H), U1.3 (B), U3.5 (2B), U8.4 (2A)
- net frame7: now also R15.1; no longer T4.5 (COLLECTOR), T4.6 (COLLECTOR), U1.11 (G), U1.4 (C), U2.3 (F), U8.1 (1A), U8.5 (2B)
- net frame8: now also R16.1; no longer T4.7 (COLLECTOR), T4.8 (COLLECTOR), U1.10 (F), U1.5 (D), U2.4 (E), U2.8 (A), U8.13 (4B), U8.2 (1B)
- net frame9: now also R17.1; no longer T5.5 (COLLECTOR), T5.6 (COLLECTOR), U2.2 (B), U2.5 (D), U6.10 (3B), U8.12 (4A)
- new net 012or13: R33.2, U3.8 (3Y)
- new net 013or14: R34.2, U6.3 (1Y)
- new net 014or15: R35.2, U6.6 (2Y)
- new net 015or16: R37.2, U6.11 (4Y)
- new net 016or1: R31.2, U2.10 (L)
- new net 03or4: R25.2, U3.3 (1Y)
- new net 04or5: R30.2, U3.11 (4Y)
- new net 05or6: R27.2, U3.6 (2Y)
- new net 05or6or7or8: R26.2, U1.1 (J)
- new net 06or7: R40.2, U8.6 (2Y)
- new net 06or7or8: R29.2, U1.13 (K)
- new net 07or8: R36.2, U8.3 (1Y)
- new net 07or8or9: R28.2, U2.6 (K)
- new net 08or9: R39.2, U8.11 (4Y)
- new net 08or9or10: R32.2, U2.9 (J)
- new net 09or10: R38.2, U6.8 (3Y)
- new net 0frame1: R2.2, T1.5 (COLLECTOR), T1.6 (COLLECTOR), U2.11 (I)
- new net 0frame10: R18.2, T5.7 (COLLECTOR), T5.8 (COLLECTOR), U2.1 (C), U6.9 (3A)
- new net 0frame11: R19.2, T6.5 (COLLECTOR), T6.6 (COLLECTOR)
- new net 0frame12: R20.2, T6.7 (COLLECTOR), T6.8 (COLLECTOR), U3.10 (3B)
- new net 0frame13: R21.2, T7.5 (COLLECTOR), T7.6 (COLLECTOR), U3.9 (3A), U6.1 (1A)
- new net 0frame14: R22.2, T7.7 (COLLECTOR), T7.8 (COLLECTOR), U6.2 (1B), U6.4 (2A)
- new net 0frame15: R23.2, T8.5 (COLLECTOR), T8.6 (COLLECTOR), U6.13 (4B), U6.5 (2B)
- new net 0frame16: R24.2, T8.7 (COLLECTOR), T8.8 (COLLECTOR), U2.12 (H), U6.12 (4A)
- new net 0frame2: R3.2, T1.7 (COLLECTOR), T1.8 (COLLECTOR)
- new net 0frame3: R11.2, T2.5 (COLLECTOR), T2.6 (COLLECTOR), U3.1 (1A)
- new net 0frame4: R12.2, T2.7 (COLLECTOR), T2.8 (COLLECTOR), U3.13 (4B), U3.2 (1B)
- new net 0frame5: R13.2, T3.5 (COLLECTOR), T3.6 (COLLECTOR), U1.2 (A), U3.12 (4A), U3.4 (2A)
- new net 0frame6: R14.2, T3.7 (COLLECTOR), T3.8 (COLLECTOR), U1.12 (H), U1.3 (B), U3.5 (2B), U8.4 (2A)
- new net 0frame7: R15.2, T4.5 (COLLECTOR), T4.6 (COLLECTOR), U1.11 (G), U1.4 (C), U2.3 (F), U8.1 (1A), U8.5 (2B)
- new net 0frame8: R16.2, T4.7 (COLLECTOR), T4.8 (COLLECTOR), U1.10 (F), U1.5 (D), U2.4 (E), U2.8 (A), U8.13 (4B), U8.2 (1B)
- new net 0frame9: R17.2, T5.5 (COLLECTOR), T5.6 (COLLECTOR), U2.2 (B), U2.5 (D), U6.10 (3B), U8.12 (4A)
