File: 8-frame-cap/grad-cap-pcb.kicad_pcb (KiCad board)
At the start: 2 copper layers, 378.4 x 339.4 mm, 177 parts, among them J1 B02B-XASK-1LFSN, T1 PHPT610035PKX, T2 PHPT610035PKX, T3 PHPT610035PKX, T4 PHPT610035PKX, T5 PHPT610035PKX, T6 PHPT610035PKX, T7 PHPT610035PKX, U1 MIC1557YM5-TR, U2 MC74HC73ADR2G, U3 SN74HCS238DYYR, U4 SN74AHCT32DBR, U5 SN74AHCT32DBR, U6 MC74HC73ADR2G

Commit message: updated from prototyping
- jk ff -> incrementer
- shrink to be cap size
- rename labels to match layout
Parts:
- removed C2, C4: .1uF, Capacitor_SMD:C_0603_1608Metric_Pad1.08x0.95mm_HandSolder
- removed R70, R71, R81, R82, R83, R84: 10K, Resistor_SMD:R_0603_1608Metric_Pad0.98x0.95mm_HandSolder
- removed U6: MC74HC73ADR2G, GRAD-CAP:MC74HC73ADR2G_JK-FLIPFLOP
- C1: value .68uF -> .1uF
- R69: value 270k -> CHECK VALUE
- U2: value MC74HC73ADR2G -> SN74HC163DR; footprint GRAD-CAP:MC74HC73ADR2G_JK-FLIPFLOP -> GRAD-CAP:binary counter - 74hc163
- moved G*** 365.9 mm to (787.5, 28.3)
- moved G*** 365.9 mm to (825.4, 32.2)
- moved G*** 365.9 mm to (828.0, 67.7)
- moved G*** 365.9 mm to (774.9, 66.4)
- moved G*** 365.9 mm to (839.8, 22.4)
- moved G*** 365.9 mm to (752.2, 15.9)
- moved G*** 365.9 mm to (789.3, 13.4)
- moved G*** 352.1 mm to (801.9, -11.8)
- moved U2 5.34 mm to (254.0, 362.5), turned to 90 degrees
- moved R74 0.81 mm to (257.2, 356.4)
- moved R72 0.80 mm to (253.8, 356.4)
- moved R73 0.79 mm to (255.5, 356.4)
Connections:
- R1 pad 1: /leds+mosfets/6c -> 7or8
- R10 pad 1: /leds+mosfets/6or7 -> 6or7
- R11 pad 1: /leds+mosfets/6c -> 7or8
- R12 pad 1: /leds+mosfets/1c -> 8or1
- R13 pad 1: /leds+mosfets/6or7 -> 6or7
- R14 pad 1: /leds+mosfets/6c -> 7or8
- R15 pad 1: /leds+mosfets/1c -> 8or1
- R16 pad 1: /leds+mosfets/6or7 -> 6or7
- R17 pad 1: /leds+mosfets/6c -> 7or8
- R18 pad 1: /leds+mosfets/1c -> 8or1
- R19 pad 1: /leds+mosfets/6or7 -> 6or7
- R2 pad 1: /leds+mosfets/1c -> 8or1
- R20 pad 1: /leds+mosfets/6c -> 7or8
- R21 pad 1: /leds+mosfets/4c -> 4or5
- R22 pad 1: /leds+mosfets/10c -> 5or6
- R23 pad 1: /leds+mosfets/2or3 -> 2or3
- R24 pad 1: /leds+mosfets/6c -> 7or8
- R25 pad 1: /leds+mosfets/2c -> frame1
- R26 pad 1: /leds+mosfets/2or3 -> 2or3
- R27 pad 1: /leds+mosfets/3c -> 3or4
- R28 pad 1: /leds+mosfets/2or3 -> 2or3
- R29 pad 1: /leds+mosfets/3c -> 3or4
- R3 pad 1: /leds+mosfets/1or2 -> 1or2
- R30 pad 1: /leds+mosfets/4c -> 4or5
- R31 pad 1: /leds+mosfets/1or2 -> 1or2
- R32 pad 1: /leds+mosfets/2or3 -> 2or3
- R33 pad 1: /leds+mosfets/3c -> 3or4
- R34 pad 1: /leds+mosfets/11c -> frame3
- R35 pad 1: /leds+mosfets/11c -> frame3
- R36 pad 1: /leds+mosfets/13c -> frame4
- R37 pad 1: /leds+mosfets/2c -> frame1
- R38 pad 1: /leds+mosfets/2or3 -> 2or3
- R39 pad 1: /leds+mosfets/3c -> 3or4
- R4 pad 1: /leds+mosfets/2or3 -> 2or3
- R40 pad 1: /leds+mosfets/4c -> 4or5
- R41 pad 1: /leds+mosfets/1or2 -> 1or2
- R42 pad 1: /leds+mosfets/2or3 -> 2or3
- R43 pad 1: /leds+mosfets/3c -> 3or4
- R44 pad 1: /leds+mosfets/6or7 -> 6or7
- R45 pad 1: /leds+mosfets/6c -> 7or8
- R46 pad 1: /leds+mosfets/1c -> 8or1
- R47 pad 1: /leds+mosfets/1or2 -> 1or2
- R48 pad 1: /leds+mosfets/9c -> frame2
- R49 pad 1: /leds+mosfets/11c -> frame3
- R5 pad 1: /leds+mosfets/3c -> 3or4
- R50 pad 1: /leds+mosfets/13c -> frame4
- R51 pad 1: /leds+mosfets/4c -> 4or5
- R52 pad 1: /leds+mosfets/10c -> 5or6
- R53 pad 1: /leds+mosfets/6or7 -> 6or7
- R54 pad 1: /leds+mosfets/13c -> frame4
- R55 pad 1: /leds+mosfets/4c -> 4or5
- R56 pad 1: /leds+mosfets/10c -> 5or6
- R57 pad 1: /leds+mosfets/6or7 -> 6or7
- R58 pad 1: /leds+mosfets/12c -> frame5
- R59 pad 1: /leds+mosfets/10c -> 5or6
- R6 pad 1: /leds+mosfets/4c -> 4or5
- R60 pad 1: /leds+mosfets/14c -> frame6
- R61 pad 1: /leds+mosfets/4c -> 4or5
- R62 pad 1: /leds+mosfets/10c -> 5or6
- R63 pad 1: /leds+mosfets/6or7 -> 6or7
- R64 pad 1: /leds+mosfets/13c -> frame4
- R65 pad 1: /leds+mosfets/4c -> 4or5
- R66 pad 1: /leds+mosfets/10c -> 5or6
- R67 pad 1: /leds+mosfets/6or7 -> 6or7
- R7 pad 1: /leds+mosfets/6or7 -> 6or7
- R8 pad 1: /leds+mosfets/6c -> 7or8
- R9 pad 1: /leds+mosfets/1c -> 8or1
- T1 pad 6: /2c -> frame1
- T1 pad 8: /1c -> 8or1
- T2 pad 6: /4c -> 4or5
- T2 pad 8: /3c -> 3or4
- T3 pad 6: /6c -> 7or8
- T3 pad 8: /2or3 -> 2or3
- T4 pad 6: /6or7 -> 6or7
- T4 pad 8: /1or2 -> 1or2
- T5 pad 6: /10c -> 5or6
- T5 pad 8: /9c -> frame2
- T6 pad 6: /12c -> frame5
- T6 pad 8: /11c -> frame3
- T7 pad 6: /14c -> frame6
- T7 pad 8: /13c -> frame4
- U2 pad 1: 557-PULSE -> +3.3V
- U2 pad 10: /u4-pu-r2-1 -> +3.3V
- U2 pad 11: GND -> CLOCK3
- U2 pad 12: CLOCK1 -> CLOCK2
- U2 pad 13: Net-(U2-*Q1) -> CLOCK1
- U2 pad 14: /u4-pu-r2-1 -> unconnected-(U2-QA-Pad14)
- U2 pad 2: /ff-reset1 -> 557-PULSE
- U2 pad 3: /ff-reset1 -> GND
- U2 pad 4: +3.3V -> GND
- U2 pad 5: CLOCK1 -> GND
- U2 pad 6: /ff-reset1 -> GND
- U2 pad 7: /ff-reset1 -> +3.3V
- U2 pad 8: Net-(U2-*Q1) -> GND
- U2 pad 9: CLOCK2 -> +3.3V
Routing:
- net 6or7: track 0.00 -> 597.3 mm, vias 0 -> 8
- net /leds+mosfets/6or7: track 597.3 -> 0.00 mm, vias 8 -> 0
- net 4or5: track 0.00 -> 498.6 mm, vias 0 -> 11
- net /leds+mosfets/4c: track 498.6 -> 0.00 mm, vias 11 -> 0
- net 3or4: track 0.00 -> 457.8 mm, vias 0 -> 6
- net /leds+mosfets/3c: track 457.8 -> 0.00 mm, vias 6 -> 0
- net 5or6: track 0.00 -> 455.4 mm, vias 0 -> 6
- net /leds+mosfets/10c: track 455.4 -> 0.00 mm, vias 6 -> 0
- net 2or3: track 0.00 -> 408.7 mm, vias 0 -> 2
- net /leds+mosfets/2or3: track 408.7 -> 0.00 mm, vias 2 -> 0
- net 8or1: track 0.00 -> 369.1 mm, vias 0 -> 6
- net /leds+mosfets/1c: track 369.1 -> 0.00 mm, vias 6 -> 0
- net 7or8: track 0.00 -> 365.3 mm, vias 0 -> 4
- net /leds+mosfets/6c: track 365.3 -> 0.00 mm, vias 4 -> 0
- net frame4: track 0.00 -> 299.2 mm, vias 0 -> 6
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Other:
- board size 378.4 x 339.4 mm -> 325.3 x 325.3 mm

Commit message: updated pcb
added labels for each diode
changed silkscreen to be handwriting
Parts:
- removed the G*** at (295.7, 256.6)
- removed the G*** at (254.0, 104.2)
- removed J1: B02B-XASK-1LFSN, GRAD-CAP:1X02JST
- removed R69: CHECK VALUE, Resistor_SMD:R_0603_1608Metric_Pad0.98x0.95mm_HandSolder
- added G***: LOGO, LOGO, F.Cu at (254.0, 256.6)
- added G***: LOGO, LOGO, B.Cu at (286.1, 253.3)
- added G***: LOGO, LOGO, B.Cu at (313.1, 252.7)
- added G***: LOGO, LOGO, F.Cu at (254.1, 102.3)
- added G***: LOGO, LOGO, F.Cu at (254.0, 249.4)
- added G***: LOGO, LOGO, F.Cu at (254.0, 245.2)
- added G***: LOGO, LOGO, F.Cu at (254.0, 240.4)
- added R70: 91AR1MEGLF, GRAD-CAP:1M-potentiometer, F.Cu at (240.3, 364.1)
- added S2: ON/OFF, GRAD-CAP:spdt-switch, F.Cu at (254.1, 377.8)
- added TP1: TestPoint, TestPoint:TestPoint_THTPad_D2.5mm_Drill1.2mm, B.Cu at (260.4, 375.8)
- added TP2: TestPoint, Connector_PinHeader_2.54mm:PinHeader_1x01_P2.54mm_Vertical, B.Cu at (247.6, 375.8)
- added U6: ICM7555xB, Package_SO:SOIC-8_3.9x4.9mm_P1.27mm, B.Cu at (265.9, 362.1)
- moved G*** 20.2 mm to (297.1, 236.3)
- moved R68 0.93 mm to (256.6, 372.7)
- moved C1 0.83 mm to (251.9, 372.9)
- moved U1 0.48 mm to (254.4, 369.8)
Connections:
- net /pd-mux-g2 renamed /pu-mux-g2
- R74 pad 2: GND -> +3.3V
Routing:
- net 557-PULSE: track 8.67 -> 19.2 mm, vias 0 -> 2
- net +BATT: track 0.00 -> 9.99 mm
- net Net-(U1-T/T): track 5.00 -> 13.5 mm, vias 0 -> 1
- net +3.3V: track 169.5 -> 175.0 mm, vias 19 -> 20
- net 5or6: track 455.4 -> 457.7 mm
- net unconnected-(U6-VCC-Pad8): track 0.00 -> 2.20 mm, vias 0 -> 1
- net unconnected-(U6-TRIG-Pad2): track 0.00 -> 2.20 mm, vias 0 -> 1
- net unconnected-(U6-GND-Pad1): track 0.00 -> 2.20 mm, vias 0 -> 1
- net unconnected-(U6-THRES-Pad6): track 0.00 -> 2.20 mm, vias 0 -> 1
- net unconnected-(U6-DISCH-Pad7): track 0.00 -> 2.20 mm, vias 0 -> 1
- net unconnected-(U6-CONT-Pad5): track 0.00 -> 2.20 mm, vias 0 -> 1
- net unconnected-(U6-OUT-Pad3): track 0.00 -> 2.20 mm, vias 0 -> 1
- net unconnected-(U6-~{RST}-Pad4): track 0.00 -> 2.19 mm, vias 0 -> 1
- net 2or3: track 408.7 -> 410.5 mm
- net GND: track 9.98 -> 11.5 mm, vias 81 -> 86
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Other:
- board text added: "a"
- board text added: "g"
- board text added: "r"
- board text added: "w"
- board text added: "{dblquote}do not even worry{dblquote}"
- board text added: "{dblquote}its all in your head{dblquote}"

Commit message: final push
Parts:
- removed the G*** at (839.8, 22.4)
- removed the G*** at (825.4, 32.2)
- removed the G*** at (828.0, 67.7)
- removed the G*** at (774.9, 66.4)
- removed the G*** at (297.1, 236.3)
- removed the G*** at (286.1, 253.3)
- removed the G*** at (313.1, 252.7)
- removed the G*** at (787.5, 28.3)
- removed the G*** at (752.2, 15.9)
- removed the G*** at (801.9, -11.8)
- removed the G*** at (789.3, 13.4)
- added G***: LOGO, LOGO, B.Cu at (242.0, 199.9)
- added G***: LOGO, LOGO, F.Cu at (340.7, 329.0)
- added G***: LOGO, LOGO, B.Cu at (242.2, 198.8)
- added G***: LOGO, LOGO, B.Cu at (227.3, 211.6)
- added G***: LOGO, LOGO, B.Cu at (227.6, 211.4)
- moved S2 116.5 mm to (361.5, 332.7), turned to 45 degrees
- moved TP2 115.0 mm to (355.5, 335.9), turned to 180 degrees
- moved TP1 114.9 mm to (364.3, 326.8), turned to -135 degrees
- moved C1 112.7 mm to (356.5, 330.8), turned to -135 degrees
- moved R68 112.6 mm to (359.7, 327.3), turned to -135 degrees
- moved U1 110.3 mm to (356.0, 326.9), turned to 135 degrees
- moved R70 106.5 mm to (342.0, 332.8), turned to 45 degrees
- moved D63 105.4 mm to (350.0, 127.5), turned to -157.5 degrees
- moved U6 104.9 mm to (358.7, 313.3), turned to -135 degrees
- moved U2 104.7 mm to (350.5, 321.9), turned to 135 degrees
- moved R63 101.6 mm to (344.9, 129.5), turned to 22.5 degrees
- moved R74 100.1 mm to (348.6, 315.3), turned to -45 degrees
- moved R73 100.1 mm to (347.3, 316.6), turned to -45 degrees
- moved R72 100.1 mm to (346.1, 317.8), turned to -45 degrees
- moved R75 99.4 mm to (360.0, 299.7), turned to 45 degrees
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Connections:
- R70 pad 1: 557-PULSE -> unconnected-(R70-Pad1)
- R70 pad 2: +3.3V -> 557-PULSE
Routing:
- net +3.3V: track 175.0 -> 165.4 mm
- net GND: track 11.5 -> 18.3 mm, vias 86 -> 90
- net 557-PULSE: track 19.2 -> 16.7 mm, vias 2 -> 1
- net +BATT: track 9.99 -> 10.8 mm
- net 5: track 29.0 -> 29.5 mm
- net f6or7: track 11.7 -> 11.2 mm
Other:
- board size 325.3 x 325.3 mm -> 230 x 230 mm
- rule pad_to_mask_clearance: 0.05 -> 0
- board text removed: "{dblquote}its all in your head{dblquote}"

Commit message: final push
inverters for pmos
resistors for mux
silkscreen looking fire as hell honestly
Parts:
- removed the G*** at (340.7, 329.0)
- removed the G*** at (227.3, 211.6)
- removed the R75 at (360.0, 299.7)
- added C1: .1uf, Capacitor_SMD:C_0805_2012Metric_Pad1.18x1.45mm_HandSolder, F.Cu at (236.4, 248.3)
- added C10: .1uf, Capacitor_SMD:C_0805_2012Metric_Pad1.18x1.45mm_HandSolder, B.Cu at (259.2, 211.7)
- added C11: .1uf, Capacitor_SMD:C_0805_2012Metric_Pad1.18x1.45mm_HandSolder, B.Cu at (237.2, 233.6)
- added C12: .1uf, Capacitor_SMD:C_0805_2012Metric_Pad1.18x1.45mm_HandSolder, B.Cu at (245.3, 225.0)
- added C13: .1uf, Capacitor_SMD:C_0805_2012Metric_Pad1.18x1.45mm_HandSolder, B.Cu at (248.1, 222.3)
- added C14: .1uf, Capacitor_SMD:C_0805_2012Metric_Pad1.18x1.45mm_HandSolder, B.Cu at (242.6, 227.8)
- added C15: .1uf, Capacitor_SMD:C_0805_2012Metric_Pad1.18x1.45mm_HandSolder, B.Cu at (250.8, 219.5)
- added C16: .1uf, Capacitor_SMD:C_0805_2012Metric_Pad1.18x1.45mm_HandSolder, B.Cu at (239.5, 230.7)
- added C17: .1uf, Capacitor_SMD:C_0805_2012Metric_Pad1.18x1.45mm_HandSolder, B.Cu at (228.7, 241.7)
- added C18: .1uf, Capacitor_SMD:C_0805_2012Metric_Pad1.18x1.45mm_HandSolder, B.Cu at (231.6, 238.9)
- added C19: .1uf, Capacitor_SMD:C_0805_2012Metric_Pad1.18x1.45mm_HandSolder, B.Cu at (234.3, 236.1)
- added C2: .1uf, Capacitor_SMD:C_0805_2012Metric_Pad1.18x1.45mm_HandSolder, F.Cu at (265.4, 241.3)
- added C20: .1uf, Capacitor_SMD:C_0805_2012Metric_Pad1.18x1.45mm_HandSolder, B.Cu at (226.3, 244.8)
- added C4: .1uf, Capacitor_SMD:C_0805_2012Metric_Pad1.18x1.45mm_HandSolder, F.Cu at (248.1, 236.6)
- added C5: .1uf, Capacitor_SMD:C_0805_2012Metric_Pad1.18x1.45mm_HandSolder, F.Cu at (257.7, 229.3)
- added C7: .1uf, Capacitor_SMD:C_0805_2012Metric_Pad1.18x1.45mm_HandSolder, B.Cu at (256.4, 214.0)
- added C8: .1uf, Capacitor_SMD:C_0805_2012Metric_Pad1.18x1.45mm_HandSolder, B.Cu at (262.1, 208.9)
- added C9: .1uf, Capacitor_SMD:C_0805_2012Metric_Pad1.18x1.45mm_HandSolder, B.Cu at (254.0, 217.3)
- added G***: LOGO, LOGO, F.Cu at (266.1, 234.0)
- added G***: LOGO, LOGO, B.Cu at (129.4, 121.7)
- added G***: LOGO, LOGO, B.Cu at (245.4, 207.4)
- added G***: LOGO, LOGO, B.Cu at (219.6, 233.6)
- added G***: LOGO, LOGO, B.Cu at (243.6, 207.2)
- added G***: LOGO, LOGO, B.Cu at (246.4, 206.4)
- added G***: LOGO, LOGO, B.Cu at (238.9, 210.9)
- added G***: LOGO, LOGO, B.Cu at (239.5, 211.4)
- added G***: LOGO, LOGO, B.Cu at (245.8, 200.8)
- added G***: LOGO, LOGO, B.Cu at (129.1, 122.9)
- added G***: LOGO, LOGO, B.Cu at (250.1, 200.5)
- added G***: LOGO, LOGO, F.Cu at (265.9, 233.0)
- added G***: LOGO, LOGO, F.Cu at (265.9, 233.5)
- added G***: LOGO, LOGO, B.Cu at (217.5, 235.0)
- added R71: 300, Resistor_SMD:R_0805_2012Metric_Pad1.20x1.40mm_HandSolder, B.Cu at (251.6, 224.3)
- added R73: 300, Resistor_SMD:R_0805_2012Metric_Pad1.20x1.40mm_HandSolder, B.Cu at (243.4, 232.6)
- added R74: 300, Resistor_SMD:R_0805_2012Metric_Pad1.20x1.40mm_HandSolder, B.Cu at (245.1, 230.9)
- added R78: 300, Resistor_SMD:R_0805_2012Metric_Pad1.20x1.40mm_HandSolder, B.Cu at (241.8, 234.2)
- added R79: 300, Resistor_SMD:R_0805_2012Metric_Pad1.20x1.40mm_HandSolder, B.Cu at (246.7, 229.3)
- added R80: 300, Resistor_SMD:R_0805_2012Metric_Pad1.20x1.40mm_HandSolder, B.Cu at (248.9, 237.7)
- added U1: SN74LVC1G14DCKR, GRAD-CAP:SN74LVC-INVERTER, F.Cu at (226.0, 244.3)
- added U10: SN74LVC1G14DCKR, GRAD-CAP:SN74LVC-INVERTER, F.Cu at (237.0, 233.3)
- added U11: SN74LVC1G14DCKR, GRAD-CAP:SN74LVC-INVERTER, F.Cu at (253.6, 216.7)
- added U12: SN74LVC1G14DCKR, GRAD-CAP:SN74LVC-INVERTER, F.Cu at (256.4, 214.0)
- added U13: SN74LVC1G14DCKR, GRAD-CAP:SN74LVC-INVERTER, F.Cu at (259.1, 211.2)
- added U14: SN74LVC1G14DCKR, GRAD-CAP:SN74LVC-INVERTER, F.Cu at (261.9, 208.4)
- added U2: SN74LVC1G14DCKR, GRAD-CAP:SN74LVC-INVERTER, F.Cu at (228.8, 241.6)
- added U3: SN74LVC1G14DCKR, GRAD-CAP:SN74LVC-INVERTER, F.Cu at (234.3, 236.1)
- added U4: SN74LVC1G14DCKR, GRAD-CAP:SN74LVC-INVERTER, F.Cu at (231.5, 238.8)
- added U5: SN74LVC1G14DCKR, GRAD-CAP:SN74LVC-INVERTER, F.Cu at (248.1, 222.3)
- added U7: SN74LVC1G14DCKR, GRAD-CAP:SN74LVC-INVERTER, F.Cu at (245.3, 225.0)
- added U8: SN74LVC1G14DCKR, GRAD-CAP:SN74LVC-INVERTER, F.Cu at (239.8, 230.5)
- added U9: SN74LVC1G14DCKR, GRAD-CAP:SN74LVC-INVERTER, F.Cu at (242.6, 227.8)
- C3: value .1uF -> .1uf; footprint Capacitor_SMD:C_0603_1608Metric_Pad1.08x0.95mm_HandSolder -> Capacitor_SMD:C_0805_2012Metric_Pad1.18x1.45mm_HandSolder; moved to F.Cu
- R76, R77: value 10k -> 300; footprint Resistor_SMD:R_0603_1608Metric_Pad0.98x0.95mm_HandSolder -> Resistor_SMD:R_0805_2012Metric_Pad1.20x1.40mm_HandSolder
- U6: value ICM7555xB -> SN74LVC1G14DCKR; footprint Package_SO:SOIC-8_3.9x4.9mm_P1.27mm -> GRAD-CAP:SN74LVC-INVERTER; moved to F.Cu
- moved U6 142.9 mm to (250.8, 219.5), turned to 135 degrees
- moved T3 132.0 mm to (232.5, 226.1)
- moved T4 132.0 mm to (243.7, 214.9)
- moved T6 132.0 mm to (249.2, 209.3)
- moved T1 132.0 mm to (221.3, 237.3)
- moved T7 132.0 mm to (254.8, 203.7)
- moved T5 132.0 mm to (238.1, 220.5)
- moved T2 132.0 mm to (226.9, 231.7)
- moved R76 130.6 mm to (250.0, 226.0), turned to -45 degrees
- moved R77 129.1 mm to (248.3, 227.6), turned to -45 degrees
- moved G*** 125.6 mm to (148.0, 115.7)
- moved D42 125.6 mm to (88.4, 239.3)
- moved R6 125.6 mm to (55.2, 148.5)
- moved R1 125.6 mm to (107.9, 42.2)
- moved R69 125.6 mm to (265.5, 244.3)
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- renumbered C1 to C6, D36 to D1, D24 to D10, D38 to D11, D37 to D12, D39 to D13, D57 to D14, D40 to D15, D15 to D16, D18 to D17, D23 to D18, D25 to D19, D33 to D2, D26 to D20, D41 to D21, D42 to D22, D56 to D23, D55 to D24, D60 to D25, D59 to D26, D13 to D27, D14 to D28, D27 to D29, D32 to D3, D16 to D30, D17 to D31, D22 to D32, D52 to D33, D43 to D34, D51 to D35, D58 to D36, D50 to D37, D49 to D38, D54 to D39, D34 to D4, D61 to D40, D62 to D41, D12 to D42, D11 to D43, D10 to D44, D19 to D45, D5 to D46, D6 to D47, D20 to D48, D53 to D49, D35 to D5, D47 to D50, D64 to D51, D48 to D52, D65 to D53, D63 to D54, D8 to D55, D7 to D56, D4 to D57, D21 to D58, D46 to D59, D30 to D6, D67 to D60, D66 to D61, D9 to D62, D3 to D63, D2 to D64, D45 to D65, D1 to D66, D44 to D67, D29 to D7, D28 to D8, D31 to D9, R36 to R1, R31 to R10, R57 to R11, R38 to R12, R39 to R13, R40 to R14, R26 to R15, R23 to R16, R18 to R17, R25 to R18, R24 to R19, R32 to R2, R41 to R20, R42 to R21, R43 to R22, R56 to R23, R55 to R24, R59 to R25, R60 to R26, R13 to R27, R15 to R28, R14 to R29, R33 to R3, R16 to R30, R17 to R31, R27 to R32, R22 to R33, R52 to R34, R51 to R35, R50 to R36, R58 to R37, R49 to R38, R54 to R39, R34 to R4, R61 to R40, R62 to R41, R12 to R42, R11 to R43, R10 to R44, R6 to R45, R19 to R46, R20 to R47, R53 to R48, R48 to R49, R35 to R5, R64 to R50, R63 to R51, R8 to R52, R7 to R53, R21 to R54, R4 to R55, R5 to R56, R47 to R57, R66 to R58, R65 to R59, R30 to R6, R9 to R60, R3 to R61, R46 to R62, R67 to R63, R2 to R64, R1 to R65, R45 to R66, R44 to R67, R70 to R68, R68 to R69, R29 to R7, R72 to R70, R74 to R72, R73 to R75, R28 to R8, R37 to R9, S2 to S1, T5 to T4, T4 to T5, TP2 to TP1, TP1 to TP2, U5 to U15, U2 to U16, U1 to U17, U3 to U18, U4 to U19
Connections:
- R76 pad 1: /u3-pd-3a -> Net-(U3-Y5)
- R76 pad 2: GND -> 5
- R77 pad 1: /u3-pd-3y -> Net-(U3-Y4)
- R77 pad 2: GND -> 4
- S1 pad 3: unconnected-(S2-Pad3) -> GND
- T1 pad 2: f1or8 -> Net-(U7-Y)
- T1 pad 4: 1 -> Net-(U11-Y)
- T2 pad 2: f3or4 -> Net-(U15-Y)
- T2 pad 4: f4or5 -> Net-(U18-Y)
- T3 pad 2: f2or3 -> Net-(U8-Y)
- T3 pad 4: f7or8 -> Net-(U12-Y)
- T4 pad 2: 2 -> Net-(U9-Y)
- T4 pad 4: f5or6 -> Net-(U13-Y)
- T5 pad 2: f1or2 -> Net-(U16-Y)
- T5 pad 4: f6or7 -> Net-(U19-Y)
- T6 pad 2: 3 -> Net-(U17-Y)
- T6 pad 4: 5 -> Net-(U20-Y)
- T7 pad 2: 4 -> Net-(U10-Y)
- T7 pad 4: 6 -> Net-(U14-Y)
- U18 pad 10: 5 -> Net-(U3-Y5)
- U18 pad 11: 4 -> Net-(U3-Y4)
- U18 pad 12: 3 -> Net-(U3-Y3)
- U18 pad 13: 2 -> Net-(U3-Y2)
- U18 pad 14: 1 -> Net-(U3-Y1)
- U18 pad 15: 0 -> Net-(U3-Y0)
- U18 pad 7: 7 -> Net-(U3-Y7)
- U18 pad 9: 6 -> Net-(U3-Y6)
- U19 pad 4: /u3-pd-3b -> 2
- U19 pad 5: /u3-pd-3a -> 3
- U19 pad 6: /u3-pd-3y -> f3or4
- U6 pad 1: unconnected-(U6-GND-Pad1) -> (no net)
- U6 pad 2: unconnected-(U6-TRIG-Pad2) -> f5or6
- U6 pad 3: unconnected-(U6-OUT-Pad3) -> GND
- U6 pad 4: unconnected-(U6-~{RST}-Pad4) -> Net-(U13-Y)
- U6 pad 5: unconnected-(U6-CONT-Pad5) -> +3.3V
Routing:
- net f3or4: track 0.00 -> 62.3 mm, vias 0 -> 2
- net GND: track 18.3 -> 69.0 mm, vias 90 -> 123
- net +3.3V: track 165.4 -> 204.0 mm, vias 20 -> 16
- net 2: track 23.4 -> 46.9 mm, vias 2 -> 8
- net Net-(U3-Y0): track 0.00 -> 8.82 mm, vias 0 -> 1
- net 4: track 29.9 -> 38.0 mm, vias 0 -> 4
- net Net-(U3-Y6): track 0.00 -> 8.03 mm, vias 0 -> 1
- net Net-(U3-Y7): track 0.00 -> 7.55 mm, vias 0 -> 1
- net Net-(U3-Y1): track 0.00 -> 7.01 mm, vias 0 -> 1
- net Net-(U3-Y5): track 0.00 -> 6.28 mm, vias 0 -> 1
- net 7: track 25.3 -> 19.0 mm, vias 2 -> 3
- net /u3-pd-3b: track 5.77 -> 0.00 mm, vias 1 -> 0
- net 3: track 19.4 -> 25.0 mm, vias 2 -> 1
- net 6: track 53.3 -> 58.9 mm, vias 4 -> 6
- net /u3-pd-3a: track 5.22 -> 0.00 mm, vias 1 -> 0
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Other:
- board text added: "330"
