File: 8-frame-cap/grad-cap-pcb.kicad_pcb (KiCad board)
At the start: 2 copper layers, 230 x 230 mm, 218 parts, among them T1 PHPT610035PKX, T2 PHPT610035PKX, T3 PHPT610035PKX, T4 PHPT610035PKX, T5 PHPT610035PKX, T6 PHPT610035PKX, T7 PHPT610035PKX, U1 SN74LVC1G14DCKR, U10 SN74LVC1G14DCKR, U11 SN74LVC1G14DCKR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

Commit message: final push
Routing:
- net GND: track 69.0 -> 67.2 mm, vias 123 -> 122
Changed lines of the file:
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@@
-	)
-	(segment
-		(start 267.627182 246.840198)
-		(end 267.627182 245.987849)
-		(width 0.4572)
-		(layer "F.Cu")
-		(net 1)
 	)
 	(segment
@@
 	)
 	(segment
-		(start 267.627182 245.987849)
-		(end 268.322228 245.292802)
-		(width 0.4572)
-		(layer "F.Cu")
-		(net 1)
-	)
-	(segment
 		(start 246.462024 225.235717)
 		(end 247.250447 224.447296)
@@
 		(tenting none)
 		(net 1)
-	)
-	(via
-		(at 268.322228 245.292802)
-		(size 0.6)
-		(drill 0.3)
-		(layers "F.Cu" "B.Cu")
-		(tenting none)
-		(net 1)
