File: 8-frame-cap/grad-cap-pcb.kicad_sch (KiCad schematic)
At the start: 26 parts, among them T1 PHPT610035PKX, T2 PHPT610035PKX, T3 PHPT610035PKX, T4 PHPT610035PKX, T5 PHPT610035PKX, T6 PHPT610035PKX, T7 PHPT610035PKX, U1 MIC1557YM5-TR, U2 SN74HC163DR, U3 SN74HCS238DYYR, U4 SN74AHCT32DBR, U5 SN74AHCT32DBR, U6 ICM7555xB

Commit message: final push
Parts:
- R70: footprint GRAD-CAP:1M-potentiometer -> RES3_91A_TTE
Connections:
- net +3.3V: no longer R70.2
- net 557-PULSE: now also R70.2; no longer R70.1
- no-connect marks 11 -> 12
Changed lines of the file:
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@@
 	)
 	(no_connect
+		(at 57.15 40.64)
+	)
+	(no_connect
 		(at 34.29 90.17)
 	)
@@
 	(wire
 		(pts
-			(xy 21.59 40.64) (xy 25.4 40.64)
+			(xy 59.69 38.1) (xy 57.15 38.1)
 		)
 		(stroke
@@
 	(wire
 		(pts
-			(xy 110.49 135.89) (xy 111.76 135.89)
+			(xy 21.59 40.64) (xy 25.4 40.64)
 		)
 		(stroke
@@
 	(wire
 		(pts
-			(xy 289.56 106.68) (xy 284.48 106.68)
+			(xy 110.49 135.89) (xy 111.76 135.89)
 		)
 		(stroke
@@
 	(wire
 		(pts
-			(xy 59.69 40.64) (xy 59.69 43.18)
+			(xy 289.56 106.68) (xy 284.48 106.68)
 		)
 		(stroke
@@
 	(wire
 		(pts
+			(xy 59.69 43.18) (xy 59.69 38.1)
+		)
+		(stroke
+			(width 0)
+			(type default)
+		)
+	)
+	(wire
+		(pts
 			(xy 110.49 140.97) (xy 111.76 140.97)
 		)
@@
 		)
 	)
-	(wire
-		(pts
-			(xy 57.15 40.64) (xy 57.15 38.1)
-		)
-		(stroke
-			(width 0)
-			(type default)
-		)
-	)
 	(polyline
 		(pts
@@
 	(symbol
 		(lib_id "power:+3.3V")
-		(at 59.69 40.64 0)
-		(unit 1)
-		(exclude_from_sim no)
-		(in_bom yes)
-		(on_board yes)
-		(dnp no)
-		(property "Reference" "#PWR051"
-			(at 59.69 44.45 0)
-			(effects
-				(font
-					(size 1.27 1.27)
-				)
-				(hide yes)
-			)
-		)
-		(property "Value" "+3.3V"
-			(at 59.69 36.83 0)
-			(effects
-				(font
-					(size 1.27 1.27)
-				)
-			)
-		)
-		(property "Footprint" ""
-			(at 59.69 40.64 0)
-			(effects
-				(font
-					(size 1.27 1.27)
-				)
-				(hide yes)
-			)
-		)
-		(property "Datasheet" ""
-			(at 59.69 40.64 0)
-			(effects
-				(font
-					(size 1.27 1.27)
-				)
-				(hide yes)
-			)
-		)
-		(property "Description" "Power symbol creates a global label with name \"+3.3V\""
-			(at 59.69 40.64 0)
-			(effects
-				(font
-					(size 1.27 1.27)
-				)
-				(hide yes)
-			)
-		)
-		(pin "1"
-		)
-		(instances
-			(project "grad-cap-pcb"
-				(path "/e928cd2e-687b-4f0f-a80d-e766cc3f22d6"
-					(reference "#PWR051")
-					(unit 1)
-				)
-			)
-		)
-	)
-	(symbol
-		(lib_id "power:+3.3V")
 		(at 21.59 35.56 0)
 		(unit 1)
@@
 		(fields_autoplaced yes)
 		(property "Reference" "R70"
-			(at 60.96 44.5007 90)
+			(at 60.96 45.7199 90)
 			(effects
 				(font
@@
 		)
 		(property "Value" "91AR1MEGLF"
-			(at 60.96 47.0407 90)
+			(at 60.96 48.2599 90)
 			(effects
 				(font
@@
 			)
 		)
-		(property "Footprint" "GRAD-CAP:1M-potentiometer"
+		(property "Footprint" "RES3_91A_TTE"
 			(at 57.15 40.64 0)
 			(effects

Commit message: final push
inverters for pmos
resistors for mux
silkscreen looking fire as hell honestly
Parts:
- removed R75: 10k, Resistor_SMD:R_0603_1608Metric_Pad0.98x0.95mm_HandSolder, symbol Device:R_Small_US
- removed U6: ICM7555xB, Package_SO:SOIC-8_3.9x4.9mm_P1.27mm, symbol Timer:ICM7555xB
- added C1, C10, C11, C12, C13, C14, C15, C16, C17, C18, C19, C2, C20, C4, C5, C7, C8, C9: .1uf, Capacitor_SMD:C_0805_2012Metric_Pad1.18x1.45mm_HandSolder, symbol Device:C_Small
- added R71, R73, R74, R78, R79, R80: 300, Resistor_SMD:R_0805_2012Metric_Pad1.20x1.40mm_HandSolder, symbol Device:R_Small_US
- added U1, U10, U11, U12, U13, U14, U2, U3, U4, U5, U6, U7, U8, U9: SN74LVC1G14DCKR, GRAD-CAP:SN74LVC-INVERTER, symbol SN74LVC-INVERTER:SN74LVC1G14DCKR
- C3: value .1uF -> .1uf; footprint Capacitor_SMD:C_0603_1608Metric_Pad1.08x0.95mm_HandSolder -> Capacitor_SMD:C_0805_2012Metric_Pad1.18x1.45mm_HandSolder
- R68: renamed from R70; footprint RES3_91A_TTE -> GRAD-CAP:1M-potentiometer
- R76, R77: value 10k -> 300; footprint Resistor_SMD:R_0603_1608Metric_Pad0.98x0.95mm_HandSolder -> Resistor_SMD:R_0805_2012Metric_Pad1.20x1.40mm_HandSolder
- U15: renamed from U5; footprint DB14 -> GRAD-CAP:SN74AHCT32DBR_2-INPUT-QUAD-OR
- U16: renamed from U2; footprint kicad_library:74hc163dr -> GRAD-CAP:binary counter - 74hc163
- U17: renamed from U1; footprint SOT-23-5_M5_MCH -> GRAD-CAP:MIC1557
- U19: renamed from U4; footprint DB14 -> GRAD-CAP:SN74AHCT32DBR_2-INPUT-QUAD-OR
- renumbered C1 to C6, R68 to R69, R72 to R70, R74 to R72, R73 to R75, S2 to S1, T5 to T4, T4 to T5, TP2 to TP1, TP1 to TP2, U3 to U18
Connections:
- net u3-pd-3b is gone; now on net 2: U19.4 (2A)
- net +3.3V: now also C1.1, C10.1, C11.1, C12.1, C13.1, C14.1, C15.1, C16.1, C17.1, C18.1, C19.1, C2.1, C20.1, C4.1, C5.1, C7.1, C8.1, C9.1, U1.5 (VCC), U10.5 (VCC), U11.5 (VCC), U12.5 (VCC), U13.5 (VCC), U14.5 (VCC), U2.5 (VCC), U3.5 (VCC), U4.5 (VCC), U5.5 (VCC), U6.5 (VCC), U7.5 (VCC), U8.5 (VCC), U9.5 (VCC)
- net 0: now also R78.2; no longer U18.15 (Y0)
- net 1: now also R73.2, U2.2 (A); no longer T1.4 (BASE), U18.14 (Y1)
- net 2: now also R74.2, U5.2 (A); no longer T4.2 (BASE), U18.13 (Y2)
- net 3: now also U19.5 (2B), R79.2, U11.2 (A); no longer T6.2 (BASE), U18.12 (Y3)
- net 4: now also R77.2, U13.2 (A); no longer T7.2 (BASE), U18.11 (Y4)
- net 5: now also R76.2, U12.2 (A); no longer T6.4 (BASE), U18.10 (Y5)
- net 6: now also R71.2, U14.2 (A); no longer T7.4 (BASE), U18.9 (Y6)
- net 7: now also R80.1; no longer U18.7 (Y7)
- net GND: now also S1.3, C1.2, C10.2, C11.2, C12.2, C13.2, C14.2, C15.2, C16.2, C17.2, C18.2, C19.2, C2.2, C20.2, C4.2, C5.2, C7.2, C8.2, C9.2, U1.3 (GND), U10.3 (GND), U11.3 (GND), U12.3 (GND), U13.3 (GND), U14.3 (GND), U2.3 (GND), U3.3 (GND), U4.3 (GND), U5.3 (GND), U6.3 (GND), U7.3 (GND), U8.3 (GND), U9.3 (GND); no longer R76.2, R77.2
- net f1or2: now also U9.2 (A); no longer T5.2 (BASE)
- net f1or8: now also U1.2 (A); no longer T1.2 (BASE)
- net f2or3: now also U10.2 (A); no longer T3.2 (BASE)
- net f3or4: now also U19.6 (2Y), U4.2 (A); no longer T2.2 (BASE)
- net f4or5: now also U3.2 (A); no longer T2.4 (BASE)
- net f5or6: now also U6.2 (A); no longer T4.4 (BASE)
- net f6or7: now also U7.2 (A); no longer T5.4 (BASE)
- net f7or8: now also U8.2 (A); no longer T3.4 (BASE)
- net u3-pd-3a: no longer names the net of R76.1
- net u3-pd-3a: now also U18.10 (Y5); no longer U19.5 (2B)
- net u3-pd-3y: no longer names the net of R77.1
- net u3-pd-3y: now also U18.11 (Y4); no longer U19.6 (2Y)
- new net: R78.1, U18.15 (Y0)
- new net: T1.2 (BASE), U1.4 (Y)
- new net: T1.4 (BASE), U2.4 (Y)
- new net: T3.2 (BASE), U10.4 (Y)
- new net: T3.4 (BASE), U8.4 (Y)
- new net: T2.2 (BASE), U4.4 (Y)
- new net: T2.4 (BASE), U3.4 (Y)
- new net: T6.4 (BASE), U12.4 (Y)
- new net: R74.1, U18.13 (Y2)
- new net: R79.1, U18.12 (Y3)
- new net: R73.1, U18.14 (Y1)
- new net: R80.2, U18.7 (Y7)
- new net: R71.1, U18.9 (Y6)
- new net: T4.2 (BASE), U5.4 (Y)
- new net: T4.4 (BASE), U6.4 (Y)
- new net: T5.2 (BASE), U9.4 (Y)
- new net: T6.2 (BASE), U11.4 (Y)
- new net: T7.4 (BASE), U14.4 (Y)
- new net: T5.4 (BASE), U7.4 (Y)
- new net: T7.2 (BASE), U13.4 (Y)
- no-connect marks 12 -> 3
Other:
- moved on the sheet: T1, T2, T3, T4, T5, T6, T7

Commit message: final push
Connections:
- net GND: no longer S1.3
Changed lines of the file:
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@@
-	)
-	(symbol
-		(lib_id "power:GND")
-		(at 67.31 189.23 0)
-		(unit 1)
-		(exclude_from_sim no)
-		(in_bom yes)
-		(on_board yes)
-		(dnp no)
-		(fields_autoplaced yes)
-		(property "Reference" "#PWR026"
-			(at 67.31 195.58 0)
-			(effects
-				(font
-					(size 1.27 1.27)
-				)
-				(hide yes)
-			)
-		)
-		(property "Value" "GND"
-			(at 67.31 194.31 0)
-			(effects
-				(font
-					(size 1.27 1.27)
-				)
-			)
-		)
-		(property "Footprint" ""
-			(at 67.31 189.23 0)
-			(effects
-				(font
-					(size 1.27 1.27)
-				)
-				(hide yes)
-			)
-		)
-		(property "Datasheet" ""
-			(at 67.31 189.23 0)
-			(effects
-				(font
-					(size 1.27 1.27)
-				)
-				(hide yes)
-			)
-		)
-		(property "Description" "Power symbol creates a global label with name \"GND\" , ground"
-			(at 67.31 189.23 0)
-			(effects
-				(font
-					(size 1.27 1.27)
-				)
-				(hide yes)
-			)
-		)
-		(pin "1"
-		)
-		(instances
-			(project "grad-cap-pcb"
-				(path "/e928cd2e-687b-4f0f-a80d-e766cc3f22d6"
-					(reference "#PWR026")
-					(unit 1)
-				)
-			)
-		)
 	)
 	(symbol
